File: Miasma_IO_smd/Miasma_IO_smd.kicad_pcb (KiCad board)
At the start: 2 copper layers, 99.1 x 99.1 mm, 137 parts, among them P1 CONN_01X12, P2 CONN_01X10, P3 CONN_01X10, P4 CONN_01X12, P5 Conn_01x02, P6 Conn_01x02, P7 CONN_01X01, Q1 MMBT3904, Q2 MMBT3904, Q3 MMBT3904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

Commit message: Added through-hole footprints for C7/C8 (polypropylene timing caps)
Other:
- board text added: "ON=Auto Cyc OFF=Trig Req"
Changed lines of the file:
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@@
   (general
     (thickness 1.6)
-    (drawings 10)
+    (drawings 12)
     (tracks 906)
     (zones 0)
@@
       (drillshape 0)
       (scaleselection 1)
-      (outputdirectory "BOM and CPL/"))
+      (outputdirectory "Gerbers/"))
   )
   (net 0 "")
@@
     )
   )
+  (gr_text "ON=Auto Cyc\nOFF=Trig Req" (at 162.5 119) (layer B.SilkS)
+    (effects (font (size 1.5 1.5) (thickness 0.3)) (justify mirror))
+  )
+  (gr_text "ON=Auto Cyc\nOFF=Trig Req" (at 129.5 119) (layer B.SilkS)
+    (effects (font (size 1.5 1.5) (thickness 0.3)) (justify mirror))
+  )
   (gr_arc (start 99.06 152.4) (end 99.06 154.94) (angle 90) (layer Edge.Cuts) (width 0.1))
